Commit message: Convert franka_config to demo3

File: urdf/environment.xacro (robot description, xacro)
@@ -4,4 +4,7 @@
   <material name="light_gray">
     <color rgba="0.7 0.7 0.7 1"/>
+  </material>
+  <material name="red">
+    <color rgba="1.0 0.1 0.1 1"/>
   </material>
   <link name="workcell_base">
@@ -55,3 +58,23 @@
   </joint>
 </xacro:macro>
+<xacro:macro name="cube" params="parent_link *location">
+<link name="cube">
+  <visual>
+    <geometry>
+      <mesh filename="package://franka_config/meshes/10_20Prism.STL"/>
+    </geometry>
+    <material name="red"/>
+  </visual>
+  <collision name="cube_collision">
+  <geometry>
+    <mesh filename="package://franka_config/meshes/10_20Prism.STL"/>
+  </geometry>
+  </collision>
+</link>
+<joint name="cube_joint" type ="fixed">
+  <xacro:insert_block name="location" />
+  <parent link="${parent_link}"/>
+  <child link="cube"/>
+</joint>
+</xacro:macro>
 </robot>

File: urdf/robot.urdf.xacro (robot description, xacro)
@@ -5,11 +5,15 @@
     <link name="base_link"/>
     <!-- Include robot -->
-    <xacro:include filename="$(find franka_config)/urdf/panda_arm.xacro"/>
+    <xacro:include filename="$(find demo3_support)/urdf/panda_arm.xacro"/>
     <xacro:panda_arm connected_to="base_link"/>
     <!-- Include workcell (creates joint from world to workcell_base)-->
-    <xacro:include filename="$(find franka_config)/urdf/environment.xacro"/>
+    <xacro:include filename="$(find demo3_support)/urdf/environment.xacro"/>
     <xacro:workcell parent_link="world" >
         <origin xyz="0.0 0.0 0.77153" rpy="0 0 0"/>
     </xacro:workcell >
+    <xacro:include filename="$(find demo3_support)/urdf/environment.xacro"/>
+    <xacro:cube parent_link="workcell_base" >
+        <origin xyz="0.15 0.4 0.1" rpy="0 0 0"/>
+    </xacro:cube >
     <!-- Create joints -->
     <joint name="workcell_base_to_base" type="fixed">
