Commit message: More demo3_support name changes

File: urdf/demo3.urdf (robot description, URDF)
Before this commit: robot robot, 13 links, 12 joints
Links:
- link cube: geometry collision mesh filename=package://demo3_support/meshes/10_20Prism.STL; visual mesh filename=package://demo3_support/meshes/10_20Prism.STL
- link panda_link0: geometry collision mesh filename=package://demo3_support/meshes/collision/link0.stl; visual mesh filename=package://demo3_support/meshes/visual/link0.dae
- link panda_link1: geometry collision mesh filename=package://demo3_support/meshes/collision/link1.stl; visual mesh filename=package://demo3_support/meshes/visual/link1.dae
- link panda_link2: geometry collision mesh filename=package://demo3_support/meshes/collision/link2.stl; visual mesh filename=package://demo3_support/meshes/visual/link2.dae
- link panda_link3: geometry collision mesh filename=package://demo3_support/meshes/collision/link3.stl; visual mesh filename=package://demo3_support/meshes/visual/link3.dae
- link panda_link4: geometry collision mesh filename=package://demo3_support/meshes/collision/link4.stl; visual mesh filename=package://demo3_support/meshes/visual/link4.dae
- link panda_link5: geometry collision mesh filename=package://demo3_support/meshes/collision/link5.stl; visual mesh filename=package://demo3_support/meshes/visual/link5.dae
- link panda_link6: geometry collision mesh filename=package://demo3_support/meshes/collision/link6.stl; visual mesh filename=package://demo3_support/meshes/visual/link6.dae
- link panda_link7: geometry collision mesh filename=package://demo3_support/meshes/collision/link7.stl; visual mesh filename=package://demo3_support/meshes/visual/link7.dae
- link workcell_base: geometry collision box size=0.1 0.1 1.25; collision box size=0.1 0.1 1.25

File: urdf/environment.xacro (robot description, xacro)
@@ -11,5 +11,5 @@
     <visual>
       <geometry>
-        <mesh filename="package://franka_config/meshes/workcell.STL"/>
+        <mesh filename="package://demo3_support/meshes/workcell.STL"/>
       </geometry>
       <material name="light_gray"/>
@@ -62,5 +62,5 @@
   <visual>
     <geometry>
-      <mesh filename="package://franka_config/meshes/10_20Prism.STL"/>
+      <mesh filename="package://demo3_support/meshes/10_20Prism.STL"/>
     </geometry>
     <material name="red"/>
@@ -68,5 +68,5 @@
   <collision name="cube_collision">
   <geometry>
-    <mesh filename="package://franka_config/meshes/10_20Prism.STL"/>
+    <mesh filename="package://demo3_support/meshes/10_20Prism.STL"/>
   </geometry>
   </collision>

File: urdf/panda_arm.xacro (robot description, xacro)
@@ -1,5 +1,5 @@
 <?xml version='1.0' encoding='utf-8'?>
 <robot xmlns:xacro="http://www.ros.org/wiki/xacro" name="panda">
-  <xacro:macro name="panda_arm" params="arm_id:='panda' description_pkg:='franka_config' connected_to:='' xyz:='0 0 0' rpy:='0 0 0'">
+  <xacro:macro name="panda_arm" params="arm_id:='panda' description_pkg:='demo3_support' connected_to:='' xyz:='0 0 0' rpy:='0 0 0'">
     <xacro:unless value="${not connected_to}">
       <joint name="${arm_id}_joint_${connected_to}" type="fixed">

Commit message: Remove box from URDF
Changed the way that the box is added in sensor simulator. This was always meant to be temporary

File: urdf/demo3.urdf (robot description, URDF)
Before this commit: robot robot, 13 links, 12 joints
Links:
- removed link cube
Joints:
- removed joint cube_joint

File: urdf/environment.xacro (robot description, xacro)
@@ -58,23 +58,4 @@
   </joint>
 </xacro:macro>
-<xacro:macro name="cube" params="parent_link *location">
-<link name="cube">
-  <visual>
-    <geometry>
-      <mesh filename="package://demo3_support/meshes/10_20Prism.STL"/>
-    </geometry>
-    <material name="red"/>
-  </visual>
-  <collision name="cube_collision">
-  <geometry>
-    <mesh filename="package://demo3_support/meshes/10_20Prism.STL"/>
-  </geometry>
-  </collision>
-</link>
-<joint name="cube_joint" type ="fixed">
-  <xacro:insert_block name="location" />
-  <parent link="${parent_link}"/>
-  <child link="cube"/>
-</joint>
 </xacro:macro>
 </robot>
